File: PCB/Padderwadder.kicad_pcb (KiCad board)
At the start: 2 copper layers, 57.5 x 41.5 mm, 5 parts, among them J1 OLED_128x32, SW3 SW_Push, SW4 SW_Push, SW5 SW_Push, U1 MOUDLE-SEEEDUINO-XIAO

Commit message: Updated PCB
Other:
- board text removed: ":)"

Commit message: Addition of rotary encoder
Parts:
- added SW1: RotaryEncoder_Switch, Rotary_Encoder:RotaryEncoder_Alps_EC11E-Switch_Vertical_H20mm, F.Cu at (155.2, 101.0)
- moved J1 13.5 mm to (115.0, 97.5)
Connections:
- U1 pad 3: unconnected-(U1-PA10_A2_D2-Pad3) -> Net-(U1-PA10_A2_D2)
- U1 pad 4: unconnected-(U1-PA11_A3_D3-Pad4) -> Net-(U1-PA11_A3_D3)
- U1 pad 7: unconnected-(U1-PB08_A6_D6_TX-Pad7) -> Net-(U1-PB08_A6_D6_TX)
Routing:
- net +3.3V: track 7.38 -> 46.7 mm
- net Net-(J1-SCL): track 23.6 -> 58.2 mm
- net Net-(U1-PB08_A6_D6_TX): track 0.00 -> 20.5 mm
- net GND: track 92.9 -> 110.9 mm
- net Net-(J1-SDA): track 23.6 -> 36.7 mm
- net Net-(U1-PA10_A2_D2): track 0.00 -> 10.3 mm
- net Net-(U1-PA11_A3_D3): track 0.00 -> 4.92 mm
